File: 2024KASAboard/2024KASAboard.kicad_sch (KiCad schematic)
At the start: 2 parts, among them U1 Pico, U2 BME280

Commit message: orange
Connections:
- net at U2.3 (CSB): now also U1.25 (GPIO19)
Changed lines of the file:
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@@
+	(wire
+		(pts
+			(xy 153.67 97.79) (xy 209.55 97.79)
+		)
+		(stroke
+			(width 0)
+			(type default)
+		)
+	)
 	(wire
 		(pts
@@
 		)
 		(stroke
+			(width 0)
+			(type default)
+		)
+	)
+	(wire
+		(pts
+			(xy 209.55 78.74) (xy 209.55 97.79)
+		)
+		(stroke

Commit message: add-wire
Connections:
- net at U1.1 (GPIO0): now also U1.38 (GND)
- net at U1.34 (GPIO28_ADC2): now also U1.40 (VBUS)
Changed lines of the file:
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@@
+	(wire
+		(pts
+			(xy 148.59 54.61) (xy 118.11 54.61)
+		)
+		(stroke
+			(width 0)
+			(type default)
+		)
+	)
 	(wire
 		(pts
@@
 	(wire
 		(pts
+			(xy 153.67 74.93) (xy 182.88 74.93)
+		)
+		(stroke
+			(width 0)
+			(type default)
+		)
+	)
+	(wire
+		(pts
 			(xy 167.64 69.85) (xy 153.67 69.85)
 		)
@@
 	(wire
 		(pts
+			(xy 182.88 59.69) (xy 153.67 59.69)
+		)
+		(stroke
+			(width 0)
+			(type default)
+		)
+	)
+	(wire
+		(pts
 			(xy 153.67 97.79) (xy 209.55 97.79)
+		)
+		(stroke
+			(width 0)
+			(type default)
+		)
+	)
+	(wire
+		(pts
+			(xy 182.88 74.93) (xy 182.88 59.69)
+		)
+		(stroke
+			(width 0)
+			(type default)
+		)
+	)
+	(wire
+		(pts
+			(xy 148.59 64.77) (xy 148.59 54.61)
 		)
 		(stroke
@@
 	(wire
 		(pts
+			(xy 118.11 54.61) (xy 118.11 59.69)
+		)
+		(stroke
+			(width 0)
+			(type default)
+		)
+	)
+	(wire
+		(pts
 			(xy 209.55 78.74) (xy 209.55 97.79)
 		)
 		(stroke
+			(width 0)
+			(type default)
+		)
+	)
+	(wire
+		(pts
+			(xy 153.67 64.77) (xy 148.59 64.77)
+		)
+		(stroke
