File: 2024KASAboard/_autosave-2024KASAboard.kicad_sch (KiCad schematic)
At the start: 2 parts, among them U1 Pico, U2 BME280

Commit message: board_and_code
ボードの修正とプログラムの追加
Connections:
- net at U1.34 (GPIO28_ADC2): no longer U1.40 (VBUS)
Other:
- note added: "I2C0_SDA(pico)-SDI(bme)"
- moved on the sheet: U2
Changed lines of the file:
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@@
 	(wire
 		(pts
-			(xy 153.67 105.41) (xy 217.17 105.41)
+			(xy 153.67 105.41) (xy 190.5 105.41)
 		)
 		(stroke
@@
 	(wire
 		(pts
-			(xy 217.17 105.41) (xy 217.17 78.74)
+			(xy 190.5 105.41) (xy 190.5 83.82)
 		)
 		(stroke
@@
 	(wire
 		(pts
-			(xy 204.47 78.74) (xy 167.64 78.74)
-		)
-		(stroke
-			(width 0)
-			(type default)
-		)
-	)
-	(wire
-		(pts
-			(xy 153.67 74.93) (xy 182.88 74.93)
+			(xy 177.8 83.82) (xy 167.64 83.82)
 		)
 		(stroke
@@
 	(wire
 		(pts
-			(xy 182.88 59.69) (xy 153.67 59.69)
+			(xy 153.67 97.79) (xy 182.88 97.79)
 		)
 		(stroke
@@
 	(wire
 		(pts
-			(xy 153.67 97.79) (xy 209.55 97.79)
+			(xy 180.34 83.82) (xy 180.34 90.17)
 		)
 		(stroke
@@
 	(wire
 		(pts
-			(xy 182.88 74.93) (xy 182.88 59.69)
+			(xy 153.67 107.95) (xy 185.42 107.95)
 		)
 		(stroke
@@
 	(wire
 		(pts
-			(xy 207.01 78.74) (xy 207.01 90.17)
-		)
-		(stroke
-			(width 0)
-			(type default)
-		)
-	)
-	(wire
-		(pts
-			(xy 153.67 107.95) (xy 212.09 107.95)
-		)
-		(stroke
-			(width 0)
-			(type default)
-		)
-	)
-	(wire
-		(pts
-			(xy 209.55 78.74) (xy 209.55 97.79)
+			(xy 182.88 83.82) (xy 182.88 97.79)
 		)
 		(stroke
@@
 	(wire
 		(pts
-			(xy 167.64 78.74) (xy 167.64 69.85)
+			(xy 167.64 83.82) (xy 167.64 69.85)
 		)
 		(stroke
@@
 	(wire
 		(pts
-			(xy 212.09 107.95) (xy 212.09 78.74)
+			(xy 185.42 107.95) (xy 185.42 83.82)
 		)
 		(stroke
@@
 	(wire
 		(pts
-			(xy 207.01 90.17) (xy 153.67 90.17)
+			(xy 180.34 90.17) (xy 153.67 90.17)
 		)
 		(stroke
@@
 		)
 	)
+	(text "I2C0_SDA(pico)-SDI(bme)"
+		(exclude_from_sim no)
+		(at 168.148 109.982 0)
+		(effects
+			(font
+				(size 1.27 1.27)
+			)
+		)
+	)
 	(symbol
 		(lib_id "0_kasa_lib-2024-:BME280")
-		(at 210.82 72.39 0)
+		(at 184.15 77.47 0)
 		(unit 1)
 		(exclude_from_sim no)
@@
 		(fields_autoplaced yes)
 		(property "Reference" "U2"
-			(at 219.71 74.9299 0)
+			(at 193.04 80.0099 0)
 			(effects
 				(font
@@
 		)
 		(property "Value" "BME280"
-			(at 219.71 77.4699 0)
+			(at 193.04 82.5499 0)
 			(effects
 				(font
@@
 		)
 		(property "Footprint" ""
-			(at 213.36 71.12 0)
+			(at 186.69 76.2 0)
 			(effects
 				(font
@@
 		)
 		(property "Datasheet" ""
-			(at 213.36 71.12 0)
+			(at 186.69 76.2 0)
 			(effects
 				(font
@@
 		)
 		(property "Description" ""
-			(at 210.82 72.39 0)
+			(at 184.15 77.47 0)
 			(effects
 				(font
